Commit message: 接入moveit

File: src/dm_ht_controller/urdf/dm_arm.urdf (robot description, URDF)
Before this commit: robot TRLC-DK1-Follower, 9 links, 8 joints
Links:
- removed link finger_left
- removed link finger_right
- link Link1: geometry collision mesh filename=package://dm_ht_controller/urdf/meshes/Link1.stl; visual mesh filename=package://dm_ht_controller/urdf/meshes/Link1.stl
- link Link6-7: geometry collision mesh filename=package://dm_ht_controller/urdf/meshes/Link6-7.stl; visual mesh filename=package://dm_ht_controller/urdf/meshes/Link6-7.stl
- link Link_2: geometry collision mesh filename=package://dm_ht_controller/urdf/meshes/Link_2.stl; visual mesh filename=package://dm_ht_controller/urdf/meshes/Link_2.stl
- link base_link: geometry collision mesh filename=package://dm_ht_controller/urdf/meshes/base_link.stl; visual mesh filename=package://dm_ht_controller/urdf/meshes/base_link.stl
- link link1-2: geometry collision mesh filename=package://dm_ht_controller/urdf/meshes/link1-2.stl; visual mesh filename=package://dm_ht_controller/urdf/meshes/link1-2.stl
- link link4-5: geometry collision mesh filename=package://dm_ht_controller/urdf/meshes/link4-5.stl; visual mesh filename=package://dm_ht_controller/urdf/meshes/link4-5.stl
- link link5-6: geometry collision mesh filename=package://dm_ht_controller/urdf/meshes/link5-6.stl; visual mesh filename=package://dm_ht_controller/urdf/meshes/link5-6.stl
Joints:
- removed joint gripper_left
- removed joint gripper_right
- joint joint2: axis 1 0 0 -> -1 0 0; limit lower=-3.141592653589793 upper=0 effort=100 velocity=3 -> lower=0 upper=3.141592653589793 effort=100 velocity=3
