Commit message: 更新了零点

File: src/dm_arm_moveit_config/config/gazebo_TRLC-DK1-Follower.urdf (robot description, URDF)
Before this commit: robot TRLC-DK1-Follower, 9 links, 8 joints
Links:
- removed link finger_left
- removed link finger_right
Joints:
- removed joint gripper_left
- removed joint gripper_right
- joint joint2: axis 1 0 0 -> -1 0 0; limit lower=-3.141592653589793 upper=0 effort=100 velocity=3 -> lower=-0.0349065850398 upper=3.141592653589793 effort=100 velocity=3
- joint joint3: limit lower=0 upper=4.71238898038469 effort=100 velocity=3 -> lower=-0.0698131700797 upper=4.71238898038469 effort=100 velocity=3

File: src/dm_ht_controller/urdf/dm_arm.urdf (robot description, URDF)
Before this commit: robot TRLC-DK1-Follower, 7 links, 6 joints
Joints:
- joint joint2: limit lower=0 upper=3.141592653589793 effort=100 velocity=3 -> lower=-0.0349065850398 upper=3.141592653589793 effort=100 velocity=3
- joint joint3: limit lower=0 upper=4.71238898038469 effort=100 velocity=3 -> lower=-0.0698131700797 upper=4.71238898038469 effort=100 velocity=3

Commit message: 移植原番茄机械臂控制服务器为达妙六轴机械臂控制服务器

File: src/dm_arm_moveit_config/config/gazebo_TRLC-DK1-Follower.urdf (robot description, URDF)
Before this commit: robot TRLC-DK1-Follower, 7 links, 6 joints
Links:
- added link link_tcp, mass 0.1; collision sphere radius=0.001; visual sphere radius=0.001
Joints:
- added joint joint_tcp: type fixed, parent Link6-7, child link_tcp, origin xyz=0.0 0.0 0.05 rpy=-1.5708 0 0

File: src/dm_ht_controller/urdf/dm_arm.urdf (robot description, URDF)
Before this commit: robot TRLC-DK1-Follower, 7 links, 6 joints
Links:
- added link link_tcp
Joints:
- added joint joint_tcp: type fixed, parent Link6-7, child link_tcp, origin xyz=0.0 0.0 0.0 rpy=-1.5708 0 0
