Commit message: 留存

File: src/dm_arm_description/urdf/DM-Arm-Description.urdf (robot description, URDF)
Before this commit: robot DM-Arm-Description, 12 links, 11 joints
Joints:
- joint joint2: limit lower=-0.0349065850398 upper=3.141592653589793 effort=100 velocity=3 -> lower=0.0 upper=3.141592653589793 effort=100 velocity=3
- joint joint3: limit lower=-0.0698131700797 upper=4.71238898038469 effort=100 velocity=3 -> lower=0.0 upper=4.71238898038469 effort=100 velocity=3
